File: DigitalInput.kicad_sch (KiCad schematic)
At the start: 33 parts, among them U12 PCF8574ATS, U17 PC817, U18 PIC817, U19 PIC817, U20 PIC817, U5 PC817, U6 PIC817, U7 PIC817, U8 PIC817

Commit message: ganti resistor 4K3 DI
Parts:
- removed R55, R56, R57, R58, R63, R64, R69, R70: 470, Resistor_SMD:R_0805_2012Metric, symbol Device:R
- R29, R30, R32, R34, R61, R62, R67, R68: value 470 -> 4k3
Connections:
- net at U17.1: now also R61.2
- net at U18.1: now also R62.2
- net at R34.2: now also U8.1
- net at U6.1: now also R30.2
- net at R67.2: now also U19.1
- net at R68.2: now also U20.1
- net at R29.2: now also U5.1
- net at R32.2: now also U7.1
